File: glr-pcb-template.kicad_sch (KiCad schematic)
At the start: 0 parts

Commit message: add glr-kicad-library as submodule
set some default values
Other:
- company: (none) -> Green Lion Racing
- title: (none) -> SET A TITLE AND UPDATE AUTHOR FIELDS (DOUBLE CLICK HERE)
Changed lines of the file:
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@@
 	(generator_version "9.0")
 	(paper "A4")
+	(title_block
+		(title "SET A TITLE AND UPDATE AUTHOR FIELDS (DOUBLE CLICK HERE)")
+		(date "${CURRENT_DATE}")
+		(rev "v1")
+		(company "Green Lion Racing")
+		(comment 1 "Author #1")
+		(comment 2 "Author #2")
+	)
+	(symbol
+		(lib_id "GLR_KiCad_Library:LOGO")
+		(at 259.08 173.99 0)
+		(unit 1)
+		(exclude_from_sim no)
+		(in_bom yes)
+		(on_board yes)
+		(dnp no)
+		(fields_autoplaced yes)
+		(property "Reference" "#G1"
+			(at 259.08 170.6241 0)
+			(effects
+				(font
+					(size 1.27 1.27)
+				)
+				(hide yes)
+			)
+		)
+		(property "Value" "LOGO"
+			(at 259.08 177.3559 0)
+			(effects
+				(font
+					(size 1.27 1.27)
+				)
+				(hide yes)
+			)
+		)
+		(property "Footprint" ""
+			(at 259.08 173.99 0)
+			(effects
+				(font
+					(size 1.27 1.27)
+				)
+				(hide yes)
+			)
+		)
+		(property "Datasheet" ""
+			(at 259.08 173.99 0)
+			(effects
+				(font
+					(size 1.27 1.27)
+				)
+				(hide yes)
+			)
+		)
+		(property "Description" ""
+			(at 259.08 173.99 0)
+			(effects
+				(font
+					(size 1.27 1.27)
+				)
+				(hide yes)
+			)
+		)
+		(instances
+			(project ""
+				(path "/be608b80-d1f2-4edd-b7a6-2b7cddd9f44f"
+					(reference "#G1")
+					(unit 1)
+				)
+			)
+		)
+	)
 	(sheet_instances
 		(path "/"
