File: glr-pcb-template.kicad_pcb (KiCad board)
At the start: 4 copper layers, 64 x 40 mm, 5 parts

Commit message: save comments to slikscreen
Other:
- board text added: "${COMPANY} ${TITLE} ${PROJECTNAME} ${REVISION} ${ISSUE_DATE} ${COMMENT1} ${COMMENT2} ${COMMENT3}"
- board text removed: "${COMPANY} ${TITLE} ${PROJECTNAME} ${REVISION} ${ISSUE_DATE}"
Changed lines of the file:
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@@
 		(layer "Edge.Cuts")
 	)
-	(gr_text "${COMPANY}\n${TITLE}\n${PROJECTNAME} ${REVISION}\n${ISSUE_DATE}"
-		(at 173.7 96.93 0)
+	(gr_text "${COMPANY}\n${TITLE}\n${PROJECTNAME} ${REVISION}\n${ISSUE_DATE}\n${COMMENT1}\n${COMMENT2}\n${COMMENT3}"
+		(at 173.96 90.93 0)
 		(layer "B.SilkS")
 		(effects
@@
 				(thickness 0.125)
 			)
-			(justify left bottom mirror)
+			(justify left top mirror)
 		)
 	)
